File: Projecte.kicad_sch (KiCad schematic)
At the start: 72 parts, among them K1 A161CS12VDC.64, Q1 IRLZ34N, Q3 IRLZ34N, Q4 IRLZ34N, Q5 IRLZ34N, Q7 IRLZ34N, U1 PIC18F448-IP, U2 OPA336Nx, U3 LM1117DT-5.0, U4 MCP2551-I-P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

Commit message: Layout_V2
Parts:
- removed C11, C12: 100n, Capacitor_SMD:C_0805_2012Metric, symbol Device:C
- added C17: 100n, Capacitor_SMD:C_0805_2012Metric, symbol Device:C
Connections:
- net Baixar: now also U1.5 (RA3/AN3/Vref+); no longer U1.4 (RA2/AN2/Vref-)
- net GND: now also C17.2
- net Pujar: now also U1.4 (RA2/AN2/Vref-); no longer U1.5 (RA3/AN3/Vref+)
- net VCC: now also C17.1
