File: Projecte.kicad_sch (KiCad schematic)
At the start: 71 parts, among them K1 A161CS12VDC.64, Q1 IRLZ34N, Q3 IRLZ34N, Q4 IRLZ34N, Q5 IRLZ34N, Q7 IRLZ34N, U1 PIC18F448-IP, U2 OPA336Nx, U3 LM1117DT-5.0, U4 MCP2551-I-P, U5 AMS1117-3.3, U6 PCA9306, U7 TPS63070RNMR, U8 MMC5883MA, Y1 Crystal

Commit message: Layout_Final
Parts:
- removed J_Programaci1: Conn_01x05_Pin, Connector_PinHeader_2.54mm:PinHeader_1x05_P2.54mm_Vertical, symbol Connector:Conn_01x05_Pin
- removed R10, R13, R14, R9: R, Resistor_SMD:R_0805_2012Metric, symbol Device:R
- removed U5: AMS1117-3.3, Package_TO_SOT_SMD:SOT-223-3_TabPin2, symbol Regulator_Linear:AMS1117-3.3
- removed U6: PCA9306, Library:PCA, symbol Interface:PCA9306
- removed U8: MMC5883MA, Package_LGA:LGA-16_3x3mm_P0.5mm, symbol Sensor_Magnetic:MMC5883MA
- added C1: 10u, Capacitor_SMD:C_0805_2012Metric, symbol Device:C
- added C14: 1u, Capacitor_SMD:C_0805_2012Metric, symbol Device:C
- added C2: 22u, Capacitor_SMD:C_0805_2012Metric, symbol Device:C
- added PROGRAMACIÓ1: Conn_01x06_Pin, Connector_PinHeader_2.54mm:PinHeader_1x06_P2.54mm_Vertical, symbol Connector:Conn_01x06_Pin
- added R12, R3, R5, R7: 2.7k, Resistor_SMD:R_0805_2012Metric, symbol Device:R
- added R23, R24, R6: 200k, Resistor_SMD:R_0805_2012Metric, symbol Device:R
- added U1: AMS1117-3.3, Package_TO_SOT_SMD:SOT-223-3_TabPin2, symbol Regulator_Linear:AMS1117-3.3
- added U3: PCA9306, Library:PCA, symbol Interface:PCA9306
- added U6: MMC5883MA, Package_LGA:LGA-16_3x3mm_P0.5mm, symbol Sensor_Magnetic:MMC5883MA
- C13: value 100n -> 10u
- Q1: renamed from Q7; footprint Package_TO_SOT_THT:TO-220-3_Vertical -> Library:SOT95P237X112-3N
- U8: renamed from U4; footprint Package_DIP:DIP-8_W7.62mm -> Library:SOIC127P599X175-8N
- renumbered J_Alimentació1 to 12V1, J_Botons1 to BOTONERA1, C14 to C10, C16 to C11, C8 to C12, C17 to C15, C5 to C16, C9 to C4, C4 to C5, C10 to C6, C15 to C7, C7 to C8, C6 to C9, ConnectorCAN1 to CAN1, D8 to D1, D6 to D2, DPM+2 to DPM+1, DPM+1 to DPM+2, DPM-2 to DPM-1, J_mOTOR1 to MOTOR1, Q4 to Q2, Q5 to Q3, Q1 to Q4, Q3 to Q5, R11 to R1, R22 to R10, R15 to R11, R8 to R13, R19 to R14, R17 to R15, R18 to R16, R4 to R17, R16 to R18, R2 to R19, R6 to R2, R7 to R20, R3 to R21, R12 to R22, R5 to R4, R21 to R8, R20 to R9, J_Rcalef1 to R_CALEFACTABLE1, U7 to U2, U3 to U4, U1 to U5, U2 to U7, Conector_USART1 to USART1, J_Sensor_Prox1 to s.PROXIMITAT1
Connections:
- net Boto_Motor: now also R23.2
- net Boto_R: now also R24.2
- net GND: now also C1.2, C14.2, C2.2, PROGRAMACIÓ1.3 (Pin_3), R23.1, R24.1, U1.1 (GND), U3.1 (GND), U6.11 (GND), U6.15 (INT), U6.9 (GND)
- net PGC: now also PROGRAMACIÓ1.5 (Pin_5)
- net PGD: now also PROGRAMACIÓ1.4 (Pin_4)
- net SCL: now also R7.1, U3.6 (SCL2)
- net SCL_S: now also R5.1, U3.3 (SCL1), U6.1 (SCL); no longer U5.21 (C2IN+/PSP2/RD2)
- net SDA: now also R12.1, U3.5 (SDA2)
- net SDA_S: now also R3.1, U3.4 (SDA1), U6.16 (SDA); no longer U5.20 (C1IN-/PSP1/RD1)
- net VCC: now also C1.1, PROGRAMACIÓ1.2 (Pin_2), R12.2, R6.1, R7.2, U1.3 (VI), U3.7 (VREF2); no longer C13.1
- net Vcc_3.3V: now also C14.1, C2.1, R3.2, R5.2, U1.2 (VO), U3.2 (VREF1), U6.13 (VDDIO), U6.2 (VDD)
- net Vpp: now also PROGRAMACIÓ1.1 (Pin_1)
- new net: C13.1, U6.10 (CAP)
- new net: R6.2, U3.8 (EN)
- no-connect marks 23 -> 25
Other:
- note added: "resistencies pull down"
- note removed: "Adaptador de nivell lògic per bus i2c del micro al sensor hall"
- note removed: "Coses ha canviar: poscicions al micro de les senyals, alimentació, capacitats desacoplamet Sens hall huella micro."
- moved on the sheet: BOTONERA1, C10, C11, C4, C6, C7, D1, DPA1, DR1, DR2, K1, L1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

Commit message: push_final
Parts:
- C1, C10, C11, C12, C13, C3, C4, C5, C6, C7: footprint Capacitor_SMD:C_0805_2012Metric -> Capacitor_SMD:C_0402_1005Metric
- L1: footprint Inductor_SMD:L_0805_2012Metric -> Inductor_SMD:L_1812_4532Metric
- Q1: value IRLZ34N -> IRLML2502
Changed lines of the file:
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@@
 		(polyline
 			(pts
-				(xy 284.48 85.09) (xy 257.175 85.09)
+				(xy 207.5453 12.9625) (xy 207.645 61.595)
 			)
 			(stroke
@@
 		(polyline
 			(pts
-				(xy 39.37 55.88) (xy 12.7 55.88)
+				(xy 284.48 60.96) (xy 177.8 60.96)
 			)
 			(stroke
@@
 		(polyline
 			(pts
-				(xy 39.37 55.88) (xy 39.37 154.305)
+				(xy 177.165 67.945) (xy 12.7 67.945)
 			)
 			(stroke
@@
 		(polyline
 			(pts
-				(xy 207.645 55.88) (xy 138.43 55.88)
+				(xy 284.48 85.09) (xy 257.175 85.09)
 			)
 			(stroke
@@
 		(polyline
 			(pts
-				(xy 177.165 67.945) (xy 12.7 67.945)
+				(xy 284.48 130.81) (xy 257.175 130.81)
 			)
 			(stroke
@@
 		(polyline
 			(pts
-				(xy 39.37 95.25) (xy 12.065 95.25)
+				(xy 177.165 60.96) (xy 177.165 198.12)
 			)
 			(stroke
@@
 		(polyline
 			(pts
-				(xy 284.48 130.81) (xy 257.175 130.81)
+				(xy 39.37 55.88) (xy 12.7 55.88)
 			)
 			(stroke
@@
 		(polyline
 			(pts
-				(xy 207.5453 12.9625) (xy 207.645 61.595)
+				(xy 284.48 71.12) (xy 257.175 71.12)
 			)
 			(stroke
@@
 		(polyline
 			(pts
-				(xy 284.48 71.12) (xy 257.175 71.12)
+				(xy 207.645 55.88) (xy 138.43 55.88)
 			)
 			(stroke
@@
 		(polyline
 			(pts
-				(xy 177.165 60.96) (xy 177.165 198.12)
+				(xy 39.37 55.88) (xy 39.37 154.305)
 			)
 			(stroke
@@
 		(polyline
 			(pts
-				(xy 284.48 157.48) (xy 257.175 157.48)
+				(xy 39.37 95.25) (xy 12.065 95.25)
 			)
 			(stroke
@@
 		(polyline
 			(pts
-				(xy 39.0524 117.475) (xy 11.7474 117.475)
+				(xy 284.48 105.41) (xy 257.175 105.41)
 			)
 			(stroke
@@
 		(polyline
 			(pts
-				(xy 138.43 12.7) (xy 138.43 67.945)
+				(xy 176.53 154.94) (xy 12.065 154.94)
 			)
 			(stroke
@@
 		(polyline
 			(pts
-				(xy 176.53 154.94) (xy 12.065 154.94)
+				(xy 39.0524 117.475) (xy 11.7474 117.475)
 			)
 			(stroke
@@
 		(polyline
 			(pts
-				(xy 284.48 105.41) (xy 257.175 105.41)
+				(xy 284.48 157.48) (xy 257.175 157.48)
 			)
 			(stroke
@@
 		(polyline
 			(pts
-				(xy 284.48 60.96) (xy 177.8 60.96)
+				(xy 138.43 12.7) (xy 138.43 67.945)
 			)
 			(stroke
@@
 			)
 		)
-		(property "Footprint" "Capacitor_SMD:C_0805_2012Metric"
+		(property "Footprint" "Capacitor_SMD:C_0402_1005Metric"
 			(at 91.1352 38.1 0)
 			(effects
@@
 			)
 		)
-		(property "Footprint" "Capacitor_SMD:C_0805_2012Metric"
+		(property "Footprint" "Capacitor_SMD:C_0402_1005Metric"
 			(at 44.1452 55.88 0)
 			(effects
@@
 			)
 		)
-		(property "Value" "IRLZ34N"
+		(property "Value" "IRLML2502"
 			(at 191.516 29.972 0)
 			(effects
@@
 			)
 		)
-		(property "Footprint" "Capacitor_SMD:C_0805_2012Metric"
+		(property "Footprint" "Capacitor_SMD:C_0402_1005Metric"
 			(at 20.0152 43.18 0)
 			(effects
@@
 			)
 		)
-		(property "Footprint" "Capacitor_SMD:C_0805_2012Metric"
+		(property "Footprint" "Capacitor_SMD:C_0402_1005Metric"
 			(at 56.8452 99.06 0)
 			(effects
@@
 			)
 		)
-		(property "Footprint" "Capacitor_SMD:C_0805_2012Metric"
+		(property "Footprint" "Capacitor_SMD:C_0402_1005Metric"
 			(at 131.7752 39.37 0)
 			(effects
@@
 			)
 		)
-		(property "Footprint" "Capacitor_SMD:C_0805_2012Metric"
+		(property "Footprint" "Capacitor_SMD:C_0402_1005Metric"
 			(at 45.4152 99.06 0)
 			(effects
@@
 			)
 		)
-		(property "Footprint" "Capacitor_SMD:C_0805_2012Metric"
+		(property "Footprint" "Capacitor_SMD:C_0402_1005Metric"
 			(at 111.4552 38.1 0)
 			(effects
@@
 			)
 		)
-		(property "Footprint" "Capacitor_SMD:C_0805_2012Metric"
+		(property "Footprint" "Capacitor_SMD:C_0402_1005Metric"
 			(at 18.7452 177.8 0)
 			(effects
@@
 			)
 		)
-		(property "Footprint" "Inductor_SMD:L_0805_2012Metric"
+		(property "Footprint" "Inductor_SMD:L_1812_4532Metric"
 			(at 48.26 58.42 0)
 			(effects
@@
 			)
 		)
-		(property "Footprint" "Capacitor_SMD:C_0805_2012Metric"
+		(property "Footprint" "Capacitor_SMD:C_0402_1005Metric"
 			(at 47.9552 36.83 0)
 			(effects
@@
 			)
 		)
-		(property "Footprint" "Capacitor_SMD:C_0805_2012Metric"
+		(property "Footprint" "Capacitor_SMD:C_0402_1005Metric"
 			(at 155.9052 184.15 0)
 			(effects
