File: Projecte.kicad_pcb (KiCad board)
At the start: 4 copper layers, 107.1 x 75.3 mm, 56 parts, among them K1 A161CS12VDC.64, Q1 IRLZ34N, Q3 IRLZ34N, Q4 IRLZ34N, Q5 IRLZ34N, Q7 IRLZ34N, U1 PIC18F448-IP, U2 LM358, U3 R-786.5-0.5, U4 MCP2551-I-P, U5 AMS1117-3.3, U6 TXB0108PW, U7 LM7805_TO220, U8 MMC5883MA, Y1 Crystal

Commit message: Layout
Parts:
- removed C_Prot_DC2: 0,33u, Capacitor_SMD:C_0805_2012Metric
- removed ConnectorCAN: DE9_Pins, Connector_Dsub:DSUB-9_Pins_Horizontal_P2.77x2.84mm_EdgePinOffset4.94mm_Housed_MountingHolesOffset4.94mm
- removed D7: D, Diode_THT:D_DO-41_SOD81_P10.16mm_Horizontal
- removed J_Alimentacio: Conn_01x02_Pin, Connector_PinHeader_2.54mm:PinHeader_1x02_P2.54mm_Vertical
- removed J_res: Conn_01x03_Pin, Connector_PinHeader_2.54mm:PinHeader_1x03_P2.54mm_Vertical
- added C1: 470u, Capacitor_SMD:C_0805_2012Metric, F.Cu at (112.0, 112.1)
- added C2: 20u, Capacitor_SMD:C_0805_2012Metric, F.Cu at (109.1, 126.2)
- added ConnectorCAN1: DE9_Pins, Connector_Dsub:DSUB-9_Pins_Horizontal_P2.77x2.54mm_EdgePinOffset9.40mm, F.Cu at (167.0, 130.9)
- added D1: Schttky, Diode_SMD:D_0805_2012Metric_Pad1.15x1.40mm_HandSolder, F.Cu at (115.7, 116.5)
- added J_Alimentació1: Conn_01x02_Pin, Connector_PinHeader_2.54mm:PinHeader_1x02_P2.54mm_Vertical, F.Cu at (102.6, 95.1)
- added J_Botons1: Conn_01x02_Pin, Connector_PinHeader_2.54mm:PinHeader_1x02_P2.54mm_Vertical, F.Cu at (132.7, 146.4)
- added J_Rcalef: Conn_01x02_Pin, Connector_PinHeader_2.54mm:PinHeader_1x02_P2.54mm_Vertical, F.Cu at (167.7, 57.1)
- added L1: L, Inductor_SMD:L_0805_2012Metric, F.Cu at (118.8, 116.1)
- added R1: 1k, Resistor_SMD:R_0805_2012Metric, F.Cu at (148.8, 78.7)
- added R13: R, Resistor_SMD:R_0805_2012Metric, F.Cu at (136.5, 142.0)
- added R14: R, Resistor_SMD:R_0805_2012Metric, F.Cu at (139.5, 138.0)
- added R15: R, Resistor_SMD:R_0805_2012Metric, F.Cu at (115.6, 120.5)
- added R16: 2k, Resistor_SMD:R_0805_2012Metric, F.Cu at (135.8, 82.7)
- added R17: 1k, Resistor_SMD:R_0805_2012Metric, F.Cu at (135.8, 78.2)
- added R18: 1k, Resistor_SMD:R_0805_2012Metric, F.Cu at (129.5, 72.9)
- added R19: 1k, Resistor_SMD:R_0805_2012Metric, F.Cu at (126.6, 74.5)
- added R7: 2k, Resistor_SMD:R_0805_2012Metric, F.Cu at (145.4, 78.8)
- C6, C7: moved to B.Cu
- D3, D4, D5, D6, D8: footprint Diode_THT:D_DO-41_SOD81_P10.16mm_Horizontal -> Diode_SMD:D_0805_2012Metric_Pad1.15x1.40mm_HandSolder
- R10, R9: value 10k -> R
- R_shunt1: value 0.005 -> 0.005R; footprint Resistor_SMD:R_0805_2012Metric -> Resistor_SMD:R_Shunt_Vishay_WSK2512_6332Metric_T2.21mm
- U2: value LM358 -> OPA336Nx; footprint Library:LM358 -> Package_TO_SOT_SMD:SOT-23-5
- U3: value R-786.5-0.5 -> LM2596S-3.3; footprint Converter_DCDC:Converter_DCDC_RECOM_R-78E-0.5_THT -> Package_TO_SOT_SMD:TO-263-5_TabPin3
- U6: value TXB0108PW -> PCA9306; footprint Package_SO:TSSOP-20_4.4x6.5mm_P0.65mm -> Library:PCA
- Y1: footprint Crystal:Crystal_SMD_HC49-SD -> Crystal:Crystal_HC18-U_Vertical
- moved R4 135.8 mm to (173.9, 100.1), turned to -90 degrees
- moved R3 129.9 mm to (168.8, 100.0), turned to 90 degrees
- moved R2 126.8 mm to (166.6, 100.0), turned to -90 degrees
- moved R12 124.2 mm to (171.4, 100.1), turned to -90 degrees
- moved R6 120.1 mm to (163.8, 100.0), turned to -90 degrees
- moved C6 109.3 mm to (169.1, 110.6), turned to -90 degrees
- moved R_shunt1 104.4 mm to (130.6, 79.7), turned to -90 degrees
- moved C5 102.9 mm to (164.1, 117.7), turned to -90 degrees
- moved U6 101.0 mm to (136.7, 137.0), turned to 90 degrees
- moved RMCLR1 98.6 mm to (104.2, 64.0), turned to 180 degrees
- moved D6 94.9 mm to (122.6, 74.3), turned to -90 degrees
- moved Conector_USART1 94.1 mm to (164.2, 148.5)
- moved R10 89.4 mm to (138.9, 131.8), turned to -90 degrees
- moved J_mOTOR1 88.9 mm to (103.2, 80.7), turned to 180 degrees
- moved D5 88.6 mm to (123.8, 83.0), turned to 90 degrees
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- renumbered Conector_USART to Conector_USART1, L_ON1 to DB1, L_PR1 to DR1, J_MCLR to J_MCLR1, J_Sensor_Prox to J_Sensor_Prox1, J_mOTOR to J_mOTOR1, R11 to R_ELIMINAR, SW_MCLR to SW_MCLR1
Connections:
- net /CORRENT! renamed /corrent
- net Net-(L_ON1-A) renamed /V_LED_ON
- net Net-(L_PR1-A) renamed /V_LED_XIP
- net Net-(U4-Rs) renamed /RsU4
- R10 pad 1: /Vcc -> VCC
- R10 pad 2: /apagar? -> /SDA
- R8 pad 2: unconnected-(R8-Pad2) -> GNDPWR
- R9 pad 1: /Vcc_3.3V -> VCC
- R9 pad 2: /final_carrera -> /SCL
- R_shunt1 pad 2: GNDPWR -> Net-(R18-Pad2)
- U1 pad 19: /Datos_i2c -> /SCL_S
- U1 pad 34: /apagar? -> /SDA_S
- U2 pad 2: GNDPWR -> GND
- U2 pad 3: /shunt -> Net-(U2-+)
- U2 pad 4: (no net) -> /V-s
- U2 pad 5: (no net) -> VCC
- U3 pad 3: Net-(D7-A) -> GNDPWR
- U5 pad 3: /Vcc -> VCC
- U6 pad 1: /SCL -> GND
- U6 pad 3: /SDA -> /SCL_S
- U6 pad 4: unconnected-(U6-A3-Pad4) -> /SDA_S
- U6 pad 5: unconnected-(U6-A4-Pad5) -> /SDA
- U6 pad 6: unconnected-(U6-A5-Pad6) -> /SCL
- U6 pad 7: unconnected-(U6-A6-Pad7) -> VCC
- U6 pad 8: /final_carrera -> unconnected-(U6-EN-Pad8)
- U7 pad 1: Net-(D7-A) -> /7V
- U8 pad 15: /final_carrera -> GND
- U8 pad 16: /i2c_nivellat -> /SDA_S
Routing:
- net VCC: track 0.00 -> 296.5 mm, vias 0 -> 6
- net GNDPWR: track 0.00 -> 207.5 mm, vias 0 -> 12
- net +12V: track 0.00 -> 136.2 mm
- net /Vpp: track 0.00 -> 60.9 mm, vias 0 -> 1
- net /Pujar: track 0.37 -> 58.5 mm
- net /M+: track 0.00 -> 47.5 mm
- net /SDA_S: track 0.00 -> 46.7 mm, vias 0 -> 1
- net GND: track 0.00 -> 46.4 mm, vias 0 -> 42
- net /Baixar: track 0.00 -> 45.8 mm
- net /MCLR: track 0.00 -> 44.8 mm
- net /R_on: track 0.00 -> 43.3 mm, vias 0 -> 1
- net /Canl: track 0.00 -> 36.0 mm
- net /Vcc_3.3V: track 0.00 -> 35.5 mm, vias 0 -> 2
- net /M-: track 0.00 -> 35.1 mm
- net /Canh: track 0.00 -> 31.5 mm
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- added copper zone on B.Cu, net GND
- removed copper zone on In2.Cu, net GND
- removed copper zone on In1.Cu, net VCC
Other:
- board size 107.1 x 75.3 mm -> 84 x 97.2 mm
- copper layers 4 -> 2

Commit message: Canvis_Layout
Parts:
- removed C1: 100n, Capacitor_SMD:C_0805_2012Metric
- removed C1: 470u, Capacitor_SMD:C_0805_2012Metric
- removed C2: 20u, Capacitor_SMD:C_0805_2012Metric
- removed C_Prot_DC1: 0,1u, Capacitor_SMD:C_0805_2012Metric
- removed D1: Schttky, Diode_SMD:D_0805_2012Metric_Pad1.15x1.40mm_HandSolder
- removed D3, D4, D5: D, Diode_SMD:D_0805_2012Metric_Pad1.15x1.40mm_HandSolder
- removed DB1: LED, LED_SMD:LED_0805_2012Metric_Pad1.15x1.40mm_HandSolder
- removed J_Programacio: Conn_01x05_Pin, Connector_PinHeader_2.54mm:PinHeader_1x05_P2.54mm_Vertical
- removed J_Rcalef: Conn_01x02_Pin, Connector_PinHeader_2.54mm:PinHeader_1x02_P2.54mm_Vertical
- removed R1: 1k, Resistor_SMD:R_0805_2012Metric
- removed REF** (x4): MountingHole_2.2mm_M2, MountingHole:MountingHole_2.2mm_M2
- removed R_ELIMINAR: 0, Resistor_SMD:R_0805_2012Metric
- added C10: 10u, Capacitor_SMD:C_0805_2012Metric, F.Cu at (164.2, 141.0)
- added C11: 100n, Capacitor_SMD:C_0805_2012Metric, B.Cu at (53.1, 93.0)
- added C12: 100n, Capacitor_SMD:C_0805_2012Metric, B.Cu at (53.1, 90.0)
- added C13: 100n, Capacitor_SMD:C_0805_2012Metric, B.Cu at (53.1, 87.0)
- added C14: 10u, Capacitor_SMD:C_0805_2012Metric, F.Cu at (166.9, 132.3)
- added C15: 10u, Capacitor_SMD:C_0805_2012Metric, F.Cu at (163.1, 132.3)
- added C16: 10u, Capacitor_SMD:C_0805_2012Metric, F.Cu at (169.9, 127.7)
- added C8: 10u, Capacitor_SMD:C_0805_2012Metric, B.Cu at (211.5, 107.4)
- added C9: 10u, Capacitor_SMD:C_0805_2012Metric, F.Cu at (159.9, 127.2)
- added DPA1: D, Diode_SMD:D_0805_2012Metric_Pad1.15x1.40mm_HandSolder, F.Cu at (164.2, 144.9)
- added DPA2: D, Diode_SMD:D_0805_2012Metric_Pad1.15x1.40mm_HandSolder, F.Cu at (167.1, 146.2)
- added DPM+1: D, Diode_SMD:D_0805_2012Metric_Pad1.15x1.40mm_HandSolder, F.Cu at (148.1, 114.9)
- added DPM+2: D, Diode_SMD:D_0805_2012Metric_Pad1.15x1.40mm_HandSolder, F.Cu at (133.9, 100.6)
- added DPM-2: D, Diode_SMD:D_0805_2012Metric_Pad1.15x1.40mm_HandSolder, F.Cu at (134.0, 114.6)
- added DR2: LED, LED_SMD:LED_0805_2012Metric, F.Cu at (195.6, 149.6)
- added J_Programaci1: Conn_01x05_Pin, Connector_PinHeader_2.54mm:PinHeader_1x05_P2.54mm_Vertical, F.Cu at (218.6, 98.9)
- added J_Rcalef1: Conn_01x02_Pin, Connector_PinHeader_2.54mm:PinHeader_1x02_P2.54mm_Vertical, F.Cu at (129.0, 128.9)
- added R11: 0, Resistor_SMD:R_0805_2012Metric, F.Cu at (66.7, 67.6)
- added R20: 1k, Resistor_SMD:R_0805_2012Metric, F.Cu at (95.0, 74.3)
- added R21: 1k, Resistor_SMD:R_0805_2012Metric, F.Cu at (95.0, 77.2)
- added R22: 680, Resistor_SMD:R_0805_2012Metric, F.Cu at (192.6, 149.6)
- C5: moved to B.Cu
- D6: value D -> DPM-1
- L1: value L -> 1,5u
- R15: value R -> 1k
- R5: value 200 -> 1k
- U1: footprint Package_DIP:DIP-40_W15.24mm -> Library:PIC258SMD
- U3: value LM2596S-3.3 -> LM1117DT-5.0; footprint Package_TO_SOT_SMD:TO-263-5_TabPin3 -> Package_TO_SOT_SMD:TO-252-3_TabPin2
- U7: value LM7805_TO220 -> TPS63070RNMR; footprint Package_TO_SOT_THT:TO-220-3_Vertical -> Library:TPS63070RNMR
- Y1: footprint Crystal:Crystal_HC18-U_Vertical -> Crystal:Crystal_SMD_0603-2Pin_6.0x3.5mm
- moved C6 122.7 mm to (53.0, 70.7), turned to 0 degrees
- moved C5 119.5 mm to (53.0, 73.7), turned to 0 degrees
- moved J_Botons1 119.0 mm to (246.7, 112.1), turned to 180 degrees
- moved J_Sensor_Prox1 111.2 mm to (246.9, 103.5), turned to 180 degrees
- moved U5 104.1 mm to (232.9, 122.4), turned to 180 degrees
- moved R9 90.5 mm to (225.9, 116.2)
- moved U6 89.6 mm to (224.7, 120.5), turned to 0 degrees
- moved U8 87.1 mm to (224.6, 125.1)
- moved C4 86.6 mm to (213.0, 122.1)
- moved Conector_USART1 86.0 mm to (247.0, 124.9), turned to 180 degrees
- moved R10 85.5 mm to (223.0, 116.2)
- moved RMCLR1 84.9 mm to (183.2, 94.8), turned to -90 degrees
- moved ConnectorCAN1 84.5 mm to (238.8, 86.4), turned to 180 degrees
- moved R13 83.6 mm to (216.5, 117.9)
- moved R14 82.4 mm to (219.5, 117.9), turned to 90 degrees
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Connections:
- net Net-(J_MCLR1-Pin_2) renamed /Man_CLR
- net Net-(R18-Pad2) renamed /Vs.7
- net Net-(U2-+) renamed /V+
- L1 pad 1: /V_DCDC -> /L1
- L1 pad 2: /V_DCDC' -> /L2
- R15 pad 1: /V_DCDC' -> /PG_
- R15 pad 2: /7V -> /Vouta1
- R5 pad 1: /V_LED_ON -> /PS
- R5 pad 2: VCC -> +12V
- R6 pad 2: /PGM -> /MCLR
- U1 pad 15: /Boto_Motor -> unconnected-(U1-T10S0/T1CKI/RC0-Pad15)
- U1 pad 16: /Boto_R -> unconnected-(U1-T1OSI/RC1-Pad16)
- U1 pad 19: /SCL_S -> unconnected-(U1-C1IN+/PSP0/RD0-Pad19)
- U1 pad 20: /S_entrada -> /SDA_S
- U1 pad 21: /S_sortida -> /SCL_S
- U1 pad 27: unconnected-(U1-P1A/ECCP1/PSP4/RD4-Pad27) -> /Boto_Motor
- U1 pad 28: unconnected-(U1-P1B/PSP5/RD5-Pad28) -> /Boto_R
- U1 pad 29: unconnected-(U1-P1C/PSP6/RD6-Pad29) -> /S_entrada
- U1 pad 30: unconnected-(U1-P1D/PSP7/RD7-Pad30) -> /S_sortida
- U1 pad 33: /R_on -> unconnected-(U1-RB0/INT0-Pad33)
- U1 pad 34: /SDA_S -> unconnected-(U1-RB1/INT1-Pad34)
- U1 pad 38: /PGM -> unconnected-(U1-RB5/PGM-Pad38)
- U1 pad 6: unconnected-(U1-RA4/TOCKI-Pad6) -> /R_on
- U3 pad 1: +12V -> GND
- U3 pad 2: GNDPWR -> VCC
- U3 pad 3: GNDPWR -> /Vouta1
- U5 pad 1: GNDPWR -> GND
- U7 pad 1: /7V -> /PS
- U7 pad 2: GND -> /PG_
- U7 pad 3: VCC -> /Vaux
Routing:
- net VCC: track 296.5 -> 0.00 mm, vias 6 -> 0
- net GNDPWR: track 207.5 -> 4.40 mm, vias 12 -> 0
- net +12V: track 136.2 -> 3.83 mm
- net /Vpp: track 60.9 -> 0.00 mm, vias 1 -> 0
- net /Pujar: track 58.5 -> 0.00 mm
- net /M+: track 47.5 -> 0.00 mm
- net /SDA_S: track 46.7 -> 0.00 mm, vias 1 -> 0
- net GND: track 46.4 -> 0.00 mm, vias 42 -> 0
- net /Baixar: track 45.8 -> 0.00 mm
- net /MCLR: track 44.8 -> 0.00 mm
- net /R_on: track 43.3 -> 5.58 mm, vias 1 -> 0
- net /Vcc_3.3V: track 35.5 -> 0.00 mm, vias 2 -> 0
- net /M-: track 35.1 -> 0.00 mm
- net /Canl: track 36.0 -> 3.33 mm
- net /shunt: track 31.0 -> 0.00 mm
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- added copper zone on F.Cu, net +12V
- added copper zone on F.Cu, net /Vouta1
- added copper zone on F.Cu, net GNDPWR
- removed copper zone on B.Cu, net GND
Other:
- board outline removed

Commit message: Layout_V2
Parts:
- removed C12: 100n, Capacitor_SMD:C_0805_2012Metric
- added C17: 100n, Capacitor_SMD:C_0805_2012Metric, B.Cu at (194.3, 100.4)
- added REF**: MountingHole_2.1mm, MountingHole:MountingHole_2.1mm, F.Cu at (162.5, 113.4)
- added REF**: MountingHole_2.1mm, MountingHole:MountingHole_2.1mm, F.Cu at (223.8, 124.1)
- added REF**: MountingHole_2.1mm, MountingHole:MountingHole_2.1mm, F.Cu at (221.1, 79.0)
- added REF**: MountingHole_2.1mm, MountingHole:MountingHole_2.1mm, F.Cu at (165.1, 76.8)
- C8: moved to F.Cu
- R11: moved to B.Cu
- moved C13 171.4 mm to (223.1, 109.2), turned to 90 degrees
- moved C6 165.0 mm to (211.8, 115.8)
- moved C5 154.3 mm to (205.4, 98.2), turned to -90 degrees
- moved C11 130.4 mm to (181.0, 118.0)
- moved R18 118.8 mm to (192.9, 97.3), turned to 180 degrees
- moved R16 118.0 mm to (188.9, 101.3)
- moved R19 117.7 mm to (192.9, 95.1)
- moved R17 116.2 mm to (188.9, 98.3), turned to 180 degrees
- moved R6 110.3 mm to (197.7, 89.8)
- moved R11 109.7 mm to (174.7, 86.8)
- moved DR1 101.6 mm to (196.8, 92.9), turned to 90 degrees
- moved ConnectorCAN1 81.8 mm to (163.5, 118.1), turned to 0 degrees
- moved R21 79.9 mm to (174.7, 83.4)
- moved R20 77.9 mm to (172.8, 78.2), turned to -90 degrees
- moved DR2 73.3 mm to (178.8, 78.3)
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Connections:
- U1 pad 4: /Baixar -> /Pujar
- U1 pad 5: /Pujar -> /Baixar
Routing:
- net VCC: track 0.00 -> 156.0 mm, vias 0 -> 16
- net GND: track 0.00 -> 63.0 mm, vias 0 -> 33
- net /Tx: track 0.00 -> 52.9 mm, vias 0 -> 1
- net /usart_tx: track 0.00 -> 39.8 mm
- net /usart_rx: track 0.00 -> 39.2 mm
- net +12V: track 3.83 -> 41.5 mm, vias 0 -> 2
- net /Rx: track 0.00 -> 37.6 mm, vias 0 -> 1
- net GNDPWR: track 4.40 -> 41.5 mm, vias 0 -> 14
- net /M-: track 0.00 -> 36.6 mm, vias 0 -> 2
- net /Pujar: track 0.00 -> 35.7 mm
- net /Baixar: track 0.00 -> 34.9 mm
- net /Boto_R: track 0.00 -> 34.8 mm
- net /Boto_Motor: track 0.00 -> 34.4 mm
- net /M+: track 0.00 -> 31.0 mm
- net /Vcc_3.3V: track 0.00 -> 27.0 mm, vias 0 -> 2
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- added copper zone on F.Cu, net /Vcc_3.3V
- added copper zone on B.Cu, net GND
- added copper zone on F.Cu, net GND
- added copper zone on B.Cu, net GNDPWR
- added copper zone on F.Cu, net VCC
Other:
- board outline added: 69.3 x 53.3 mm

Commit message: Push
Parts:
- moved REF** 10.8 mm to (160.9, 124.1)
- renumbered ConnectorCAN1 to ConnectorCAN
Changed lines of the file:
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@@
 	(footprint "MountingHole:MountingHole_2.1mm"
 		(layer "F.Cu")
-		(at 162.52 113.42)
+		(at 160.93 124.11)
 		(descr "Mounting Hole 2.1mm, no annular")
 		(tags "mounting hole 2.1mm no annular")
@@
 		(descr "9-pin D-Sub connector, horizontal/angled (90 deg), THT-mount, pins (male), pitch 2.77x2.54mm, pin-PCB-offset 9.4mm, see https://docs.rs-online.com/02d6/0900766b81585df2.pdf")
 		(tags "9-pin D-Sub connector horizontal angled 90deg THT pins pitch 2.77x2.54mm pin-PCB-offset 9.4mm")
-		(property "Reference" "ConnectorCAN1"
-			(at -4.38 3.245331 90)
+		(property "Reference" "ConnectorCAN"
+			(at 5.54 6.285331 180)
 			(layer "F.SilkS")
 			(effects

Commit message: Layout_Final
Parts:
- removed J_Programaci1: Conn_01x05_Pin, Connector_PinHeader_2.54mm:PinHeader_1x05_P2.54mm_Vertical
- removed the R10 at (214.8, 105.0)
- removed the R13 at (214.0, 109.0)
- removed the R14 at (211.6, 109.0)
- removed the R9 at (209.4, 109.0)
- removed the U5 at (211.9, 115.6)
- removed the U8 at (220.3, 113.3)
- added C13: 10u, Capacitor_SMD:C_0805_2012Metric, F.Cu at (224.7, 119.0)
- added C14: 1u, Capacitor_SMD:C_0805_2012Metric, F.Cu at (212.7, 127.1)
- added C2: 22u, Capacitor_SMD:C_0805_2012Metric, F.Cu at (224.8, 124.7)
- added PROGRAMACIÓ: Conn_01x06_Pin, Connector_PinHeader_2.54mm:PinHeader_1x06_P2.54mm_Vertical, F.Cu at (203.6, 88.7)
- added R12: 2.7k, Resistor_SMD:R_0805_2012Metric, F.Cu at (216.4, 104.4)
- added R23: 200k, Resistor_SMD:R_0805_2012Metric, B.Cu at (222.3, 91.2)
- added R24: 200k, Resistor_SMD:R_0805_2012Metric, B.Cu at (222.3, 88.6)
- added R3: 2.7k, Resistor_SMD:R_0805_2012Metric, F.Cu at (225.2, 114.2)
- added R5: 2.7k, Resistor_SMD:R_0805_2012Metric, F.Cu at (217.7, 114.1)
- added R6: 200k, Resistor_SMD:R_0805_2012Metric, F.Cu at (216.4, 110.2)
- added R7: 2.7k, Resistor_SMD:R_0805_2012Metric, F.Cu at (216.5, 107.7)
- added U1: AMS1117-3.3, Package_TO_SOT_SMD:SOT-223-3_TabPin2, F.Cu at (212.8, 120.7)
- added U3: PCA9306, Library:PCA, F.Cu at (221.3, 109.6)
- Q1: renamed from Q7; footprint Package_TO_SOT_THT:TO-220-3_Vertical -> Library:SOT95P237X112-3N
- R CALEFACTABLE: renamed from J_Rcalef1
- SW MCLR: renamed from SW_MCLR1
- U6: value PCA9306 -> MMC5883MA; footprint Library:PCA -> Package_LGA:LGA-16_3x3mm_P0.5mm
- U8: renamed from U4; footprint Package_DIP:DIP-8_W7.62mm -> Library:SOIC127P599X175-8N
- moved R CALEFACTABLE 37.8 mm to (159.9, 114.4), turned to 0 degrees
- moved BOTONERA 34.7 mm to (226.8, 91.2), turned to 180 degrees
- moved USART 30.7 mm to (226.8, 104.1), turned to 180 degrees
- moved R22 26.9 mm to (195.2, 116.2)
- moved CAN 25.1 mm to (188.6, 119.0)
- moved K1 24.1 mm to (172.1, 115.6), turned to 0 degrees
- moved s.PROXIMITAT 20.7 mm to (223.6, 80.2), turned to -90 degrees
- moved R17 20.5 mm to (198.8, 116.4)
- moved R19 17.5 mm to (190.9, 109.0), turned to -90 degrees
- moved R21 16.9 mm to (191.0, 112.7), turned to -90 degrees
- moved C11 15.7 mm to (195.2, 111.0), turned to 90 degrees
- moved U8 14.9 mm to (195.2, 111.0), turned to -90 degrees
- moved D1 10.1 mm to (181.7, 113.0), turned to 90 degrees
- moved U6 10.1 mm to (221.0, 118.8)
- moved R13 9.47 mm to (184.3, 113.1), turned to 90 degrees
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- renumbered J_Alimentació1 to 12V, J_Botons1 to BOTONERA, C14 to C10, C16 to C11, C8 to C12, C17 to C15, C5 to C16, C9 to C4, C4 to C5, C10 to C6, C15 to C7, C7 to C8, C6 to C9, ConnectorCAN to CAN, D8 to D1, D6 to D2, DPM+2 to DPM+1, DPM+1 to DPM+2, DPM-2 to DPM-1, J_MCLR1 to MCLR, J_mOTOR1 to MOTOR, Q4 to Q2, Q5 to Q3, Q1 to Q4, Q3 to Q5, R11 to R1, R22 to R10, R15 to R11, R8 to R13, R19 to R14, R17 to R15, R18 to R16, R4 to R17, R16 to R18, R2 to R19, R6 to R2, R7 to R20, R3 to R21, R12 to R22, R5 to R4, R21 to R8, R20 to R9, U7 to U2, U3 to U4, U1 to U5, U2 to U7, Conector_USART1 to USART, J_Sensor_Prox1 to s.PROXIMITAT
Connections:
- U5 pad 20: /SDA_S -> unconnected-(U5-C1IN-/PSP1/RD1-Pad20)
- U5 pad 21: /SCL_S -> unconnected-(U5-C2IN+/PSP2/RD2-Pad21)
- U6 pad 1: GND -> /SCL_S
- U6 pad 3: /SCL_S -> unconnected-(U6-NC-Pad3)
- U6 pad 4: /SDA_S -> unconnected-(U6-NC-Pad4)
- U6 pad 5: /SDA -> unconnected-(U6-NC-Pad5)
- U6 pad 6: /SCL -> unconnected-(U6-NC-Pad6)
- U6 pad 7: VCC -> unconnected-(U6-NC-Pad7)
Routing:
- net VCC: track 156.0 -> 109.9 mm, vias 16 -> 10
- net /Tx: track 52.9 -> 22.6 mm, vias 1 -> 2
- net /usart_tx: track 39.8 -> 13.5 mm
- net /Vcc_3.3V: track 27.0 -> 53.2 mm, vias 2 -> 0
- net /usart_rx: track 39.2 -> 14.2 mm
- net /S_entrada: track 9.42 -> 23.6 mm
- net /Rx: track 37.6 -> 25.3 mm, vias 1 -> 2
- net /Boto_Motor: track 34.4 -> 22.3 mm
- net /S_sortida: track 10.3 -> 20.9 mm
- net /Boto_R: track 34.8 -> 24.5 mm
- net /SDA_S: track 20.2 -> 10.0 mm, vias 2 -> 0
- net /PGD: track 15.4 -> 8.17 mm
- net /PGC: track 17.1 -> 10.3 mm
- net /SCL_S: track 16.8 -> 10.2 mm, vias 2 -> 0
- net /Canh: track 17.6 -> 11.1 mm
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- removed copper zone on F.Cu, net /Vcc_3.3V
Other:
- board size 69.3 x 53.3 mm -> 74.8 x 56.6 mm
- board text added: "PCB MALETERO JORDI COMAS ELENA SANS"
- board text added: "REF:"

Commit message: .
Other:
- board text added: "PCB MALETERO JORDI COMAS i ELENA SANS"
- board text removed: "PCB MALETERO JORDI COMAS ELENA SANS"
